Commit message: Fix: Rename package

File: urdf/robot.urdf.xacro (robot description, xacro)
@@ -1,4 +1,4 @@
 <?xml version = "1.0"?>
-<robot xmlns:xacro="https://www.rog.org/wiki/xacro" name="robot">
+<robot xmlns:xacro="https://www.rog.org/wiki/xacro" name="mobilerobot">
     <xacro:include filename="robot_core.xacro" />
 </robot>

File: urdf/robot_core.xacro (robot description, xacro)
@@ -13,44 +13,30 @@
         <color rgba = "0.96 0.95 0.92 1"/>
     </material>
-    <link name="base_link">
+    <!-- ========================================== -->
+    <!--         GỐC ẢO VÀ TRỌNG TÂM ROBOT          -->
+    <!-- ========================================== -->
+    <link name="base_footprint"/>
+    <link name="base_link"/>
+    <joint name="base_footprint" type="fixed">
+        <parent link="base_footprint"/>
+        <child link="base_link"/>
+        <origin xyz="0 0 0.015" rpy="0 0 0"/>
+    </joint>
+    <!-- ========================================== -->
+    <!--              Thân xe (Chasis)              -->
+    <!-- ========================================== -->
+    <link name="chasis_link">
         <visual>
-            <origin xyz="0 0 0"/>
+            <origin xyz="0 0 0.05"/>   <!-- Vị trí của tâm khối so với gốc tọa độ (trục bánh xe)-->
             <geometry>
-                <sphere radius="0.1"/>
-            </geometry>
-            <material name="c3"/>
-        </visual>
-    </link>
-    <link name="base_footprint"/>
-        <visual>
-            <origin xyz="0 0 0"/>
-            <geometry>
-                <sphere radius="0.1"/>
-            </geometry>
-            <material name="c3"/>
-        </visual>
-    </link>
-    <link name="base_link">
-        <visual>
-            <origin xyz="0 0 0"/>
-            <geometry>
-                <sphere radius="0.1"/>
-            </geometry>
-            <material name="c3"/>
-        </visual>
-    </link>
-    <joint name="tes_joint" type="fixed">
-        <parent link="base_link"/>
-        <child link="tes"/>
-        <origin xyz="-0.1 0 0"/>
-    </joint>
-    <link name="tes">
-        <visual>
-            <origin xyz="-0.5 -0.5 -0.5"/>
-            <geometry>
-                <box size="1 1 1"/>
+                <box size="0.3 0.3 0.2"/>
             </geometry>
             <material name="matcha"/>
         </visual>
     </link>
+    <joint name="chasis_base" type="fixed">
+        <parent link="base_link"/>
+        <child link="chasis_link"/>
+        <origin xyz="0 0 0.05"/>
+    </joint>
 </robot>

Commit message: Done basic URDF, no Gazebo

File: urdf/robot.urdf.xacro (robot description, xacro)
@@ -1,4 +1,4 @@
 <?xml version = "1.0"?>
-<robot xmlns:xacro="https://www.rog.org/wiki/xacro" name="mobilerobot">
+<robot xmlns:xacro="https://www.ros.org/wiki/xacro" name="robot">
     <xacro:include filename="robot_core.xacro" />
 </robot>

File: urdf/robot_core.xacro (robot description, xacro)
@@ -1,42 +1,87 @@
-<?xml version = "1.0"?>
-<robot xmlns:xacro="https://www.rog.org/wiki/xacro" name="robot">
-    <material name="red">
-        <color rgba = "0.5 0.125 0.125 1"/>
-    </material>
-    <material name="matcha">
-        <color rgba = "0.52 0.6 0.49 1"/>
-    </material>
-    <material name="c3">
-        <color rgba = "0.785 0.789 0.672 1"/>
-    </material>
-    <material name="c4">
-        <color rgba = "0.96 0.95 0.92 1"/>
-    </material>
-    <!-- ========================================== -->
-    <!--         GỐC ẢO VÀ TRỌNG TÂM ROBOT          -->
-    <!-- ========================================== -->
+<?xml version="1.0"?>
+<robot xmlns:xacro="http://www.ros.org/wiki/xacro">
+    <xacro:include filename="inertial_macros.xacro"/>
+    <material name="red"><color rgba="0.5 0.125 0.125 1"/></material>
+    <material name="matcha"><color rgba="0.52 0.6 0.49 1"/></material>
+    <material name="c3"><color rgba="0.785 0.789 0.672 1"/></material>
+    <material name="c4"><color rgba="0.96 0.95 0.92 1"/></material>
     <link name="base_footprint"/>
     <link name="base_link"/>
-    <joint name="base_footprint" type="fixed">
+    <joint name="base_footprint_joint" type="fixed">
         <parent link="base_footprint"/>
         <child link="base_link"/>
-        <origin xyz="0 0 0.015" rpy="0 0 0"/>
+        <origin xyz="0 0 0.012" rpy="0 0 0"/>
     </joint>
-    <!-- ========================================== -->
-    <!--              Thân xe (Chasis)              -->
-    <!-- ========================================== -->
     <link name="chasis_link">
         <visual>
-            <origin xyz="0 0 0.05"/>   <!-- Vị trí của tâm khối so với gốc tọa độ (trục bánh xe)-->
-            <geometry>
-                <box size="0.3 0.3 0.2"/>
-            </geometry>
+            <origin xyz="0 0 0.0425"/>
+            <geometry><box size="0.15 0.15 0.085"/></geometry>
             <material name="matcha"/>
         </visual>
+        <collision>
+            <origin xyz="0 0 0.0425"/>
+            <geometry><box size="0.15 0.15 0.085"/></geometry>
+        </collision>
+        <xacro:inertial_box mass="0.5" x="0.15" y="0.15" z="0.085">
+            <origin xyz="0 0 0.0425" rpy="0 0 0"/>
+        </xacro:inertial_box>
     </link>
     <joint name="chasis_base" type="fixed">
         <parent link="base_link"/>
         <child link="chasis_link"/>
-        <origin xyz="0 0 0.05"/>
+        <origin xyz="0 0 0"/>
     </joint>
-</robot>
+    <link name="left_wheel_link">
+        <visual>
+            <geometry><cylinder radius="0.0215" length="0.018"/></geometry>
+            <material name="c4"/>
+        </visual>
+        <collision>
+            <geometry><cylinder radius="0.0215" length="0.018"/></geometry>
+        </collision>
+        <xacro:inertial_cylinder mass="0.015" radius="0.0215" length="0.018">
+            <origin xyz="0 0 0" rpy="0 0 0"/>
+        </xacro:inertial_cylinder>
+    </link>
+    <joint name="left_wheel_base" type="continuous">
+        <parent link="base_link"/>
+        <child link="left_wheel_link"/>
+        <origin xyz="0 0.084 0.0095" rpy="${-pi/2} 0 0"/>
+        <axis xyz="0 0 1"/>
+    </joint>
+    <link name="right_wheel_link">
+        <visual>
+            <geometry><cylinder radius="0.0215" length="0.018"/></geometry>
+            <material name="c4"/>
+        </visual>
+        <collision>
+            <geometry><cylinder radius="0.0215" length="0.018"/></geometry>
+        </collision>
+        <xacro:inertial_cylinder mass="0.015" radius="0.0215" length="0.018">
+            <origin xyz="0 0 0" rpy="0 0 0"/>
+        </xacro:inertial_cylinder>
+    </link>
+    <joint name="right_wheel_base" type="continuous">
+        <parent link="base_link"/>
+        <child link="right_wheel_link"/>
+        <origin xyz="0 -0.084 0.0095" rpy="${pi/2} 0 0"/>
+        <axis xyz="0 0 -1"/>
+    </joint>
+    <link name="caster1_link">
+        <visual>
+            <geometry><sphere radius="0.006"/></geometry>
+            <material name="c3"/>
+        </visual>
+        <collision>
+            <geometry><sphere radius="0.006"/></geometry>
+        </collision>
+        <xacro:inertial_sphere mass="0.015" radius="0.006">
+            <origin xyz="0 0 0" rpy="0 0 0"/>
+        </xacro:inertial_sphere>
+    </link>
+    <joint name="caster1_base" type="fixed">
+        <parent link="base_link"/>
+        <child link="caster1_link"/>
+        <origin xyz="0.055 0.055 -0.006"/>
+    </joint>
+    </robot>
