Commit message: add Gazebo appearance to URDF and file launch test

File: urdf/robot_core.xacro (robot description, xacro)
@@ -27,4 +27,7 @@
         </xacro:inertial_box>
     </link>
+    <gazebo reference="chasis_link">
+        <material>Gazebo/Grass</material>
+    </gazebo>
     <joint name="chasis_base" type="fixed">
         <parent link="base_link"/>
@@ -44,4 +47,7 @@
         </xacro:inertial_cylinder>
     </link>
+    <gazebo reference="left_wheel_link">
+        <material>Gazebo/Ivory</material>
+    </gazebo>
     <joint name="left_wheel_base" type="continuous">
         <parent link="base_link"/>
@@ -62,4 +68,7 @@
         </xacro:inertial_cylinder>
     </link>
+    <gazebo reference="right_wheel_link">
+        <material>Gazebo/Ivory</material>
+    </gazebo>
     <joint name="right_wheel_base" type="continuous">
         <parent link="base_link"/>
@@ -80,4 +89,7 @@
         </xacro:inertial_sphere>
     </link>
+    <gazebo reference="caster1_link">
+        <material>Gazebo/Sand</material>
+    </gazebo>
     <joint name="caster1_base" type="fixed">
         <parent link="base_link"/>
@@ -85,3 +97,80 @@
         <origin xyz="0.055 0.055 -0.006"/>
     </joint>
-    </robot>
+    <link name="caster2_link">
+        <visual>
+            <geometry><sphere radius="0.006"/></geometry>
+            <material name="c3"/>
+        </visual>
+        <collision>
+            <geometry><sphere radius="0.006"/></geometry>
+        </collision>
+        <xacro:inertial_sphere mass="0.015" radius="0.006">
+            <origin xyz="0 0 0" rpy="0 0 0"/>
+        </xacro:inertial_sphere>
+    </link>
+    <gazebo reference="caster2_link">
+        <material>Gazebo/Sand</material>
+    </gazebo>
+    <joint name="caster2_base" type="fixed">
+        <parent link="base_link"/>
+        <child link="caster2_link"/>
+        <origin xyz="-0.055 0.055 -0.006"/>
+    </joint>
+    <link name="caster3_link">
+        <visual>
+            <geometry><sphere radius="0.006"/></geometry>
+            <material name="c3"/>
+        </visual>
+        <collision>
+            <geometry><sphere radius="0.006"/></geometry>
+        </collision>
+        <xacro:inertial_sphere mass="0.015" radius="0.006">
+            <origin xyz="0 0 0" rpy="0 0 0"/>
+        </xacro:inertial_sphere>
+    </link>
+    <gazebo reference="caster3_link">
+        <material>Gazebo/Sand</material>
+    </gazebo>
+    <joint name="caster3_base" type="fixed">
+        <parent link="base_link"/>
+        <child link="caster3_link"/>
+        <origin xyz="0.055 -0.055 -0.006"/>
+    </joint>
+    <link name="caster4_link">
+        <visual>
+            <geometry><sphere radius="0.006"/></geometry>
+            <material name="c3"/>
+        </visual>
+        <collision>
+            <geometry><sphere radius="0.006"/></geometry>
+        </collision>
+        <xacro:inertial_sphere mass="0.015" radius="0.006">
+            <origin xyz="0 0 0" rpy="0 0 0"/>
+        </xacro:inertial_sphere>
+    </link>
+    <gazebo reference="caster4_link">
+        <material>Gazebo/Sand</material>
+    </gazebo>
+    <joint name="caster4_base" type="fixed">
+        <parent link="base_link"/>
+        <child link="caster4_link"/>
+        <origin xyz="-0.055 -0.055 -0.006"/>
+    </joint>
+    <gazebo>
+        <plugin name="differential_drive_controller" filename="libgazebo_ros_diff_drive.so">
+            <updateRate>100</updateRate>
+            <leftJoint>left_wheel_base</leftJoint>
+            <rightJoint>right_wheel_base</rightJoint>
+            <wheelSeparation>0.168</wheelSeparation>
+            <wheelDiameter>0.043</wheelDiameter>
+            <wheelAcceleration>1.0</wheelAcceleration>
+            <wheelTorque>20</wheelTorque>
+            <commandTopic>cmd_vel</commandTopic>
+            <odometryTopic>odom</odometryTopic>
+            <odometryFrame>odom</odometryFrame>
+            <robotBaseFrame>base_footprint</robotBaseFrame>
+            <publishWheelTF>true</publishWheelTF>
+            <publishOdomTF>true</publishOdomTF>
+        </plugin>
+    </gazebo>
+</robot>
